File: EQModule/EQModule.kicad_sch (KiCad schematic)
At the start: 10 parts, among them J1 SigIn, J2 SigOut, J3 TreblePot, J4 BassPot, J5 MidPot, J6 VolPot

Commit message: Change connector footprints to contain 3D models. Make necessary PCB modifications to address errors found in the design
Parts:
- J1, J2: footprint Connector_Molex:Molex_Micro-Fit_3.0_43650-0200_1x02_P3.00mm_Horizontal -> CustomFootprints:Molex_Micro-Fit_3.0_43650-0200_1x02_P3.00mm_Horizontal
- J3, J4, J5, J6: footprint Connector_Molex:Molex_Micro-Fit_3.0_43650-0315_1x03_P3.00mm_Vertical -> CustomFootprints:Molex_Micro-Fit_3.0_43650-0315_1x03_P3.00mm_Vertical
Changed lines of the file:
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@@
       (effects (font (size 1.27 1.27)) (justify left))
     )
-    (property "Footprint" "Connector_Molex:Molex_Micro-Fit_3.0_43650-0315_1x03_P3.00mm_Vertical" (at 140.97 82.55 0)
+    (property "Footprint" "CustomFootprints:Molex_Micro-Fit_3.0_43650-0315_1x03_P3.00mm_Vertical" (at 140.97 82.55 0)
       (effects (font (size 1.27 1.27)) hide)
     )
@@
       (effects (font (size 1.27 1.27)) (justify left))
     )
-    (property "Footprint" "Connector_Molex:Molex_Micro-Fit_3.0_43650-0200_1x02_P3.00mm_Horizontal" (at 157.48 82.55 0)
+    (property "Footprint" "CustomFootprints:Molex_Micro-Fit_3.0_43650-0200_1x02_P3.00mm_Horizontal" (at 157.48 82.55 0)
       (effects (font (size 1.27 1.27)) hide)
     )
@@
       (effects (font (size 1.27 1.27)) (justify left))
     )
-    (property "Footprint" "Connector_Molex:Molex_Micro-Fit_3.0_43650-0200_1x02_P3.00mm_Horizontal" (at 114.3 95.25 0)
+    (property "Footprint" "CustomFootprints:Molex_Micro-Fit_3.0_43650-0200_1x02_P3.00mm_Horizontal" (at 114.3 95.25 0)
       (effects (font (size 1.27 1.27)) hide)
     )
@@
       (effects (font (size 1.27 1.27)) (justify left))
     )
-    (property "Footprint" "Connector_Molex:Molex_Micro-Fit_3.0_43650-0315_1x03_P3.00mm_Vertical" (at 139.7 93.98 0)
+    (property "Footprint" "CustomFootprints:Molex_Micro-Fit_3.0_43650-0315_1x03_P3.00mm_Vertical" (at 139.7 93.98 0)
       (effects (font (size 1.27 1.27)) hide)
     )
@@
       (effects (font (size 1.27 1.27)))
     )
-    (property "Footprint" "Connector_Molex:Molex_Micro-Fit_3.0_43650-0315_1x03_P3.00mm_Vertical" (at 139.7 105.41 0)
+    (property "Footprint" "CustomFootprints:Molex_Micro-Fit_3.0_43650-0315_1x03_P3.00mm_Vertical" (at 139.7 105.41 0)
       (effects (font (size 1.27 1.27)) hide)
     )
@@
       (effects (font (size 1.27 1.27)) (justify left))
     )
-    (property "Footprint" "Connector_Molex:Molex_Micro-Fit_3.0_43650-0315_1x03_P3.00mm_Vertical" (at 149.86 114.3 0)
-      (effects (font (size 1.27 1.27)) hide)
-    )
+    (property "Footprint" "CustomFootprints:Molex_Micro-Fit_3.0_43650-0315_1x03_P3.00mm_Vertical" (at 149.86 114.3 0)
+      (effects (font (size 1.27 1.27)) hide)
+    )
