File: Gain1Module/Gain1Module.kicad_sch (KiCad schematic)
At the start: 21 parts, among them J1 Low Jack, J2 High Jack, J3 HV, J4 Heater, J5 Signal, J6 Vol, U1 ECC83

Commit message: Change connector footprints to contain 3D models. Make necessary PCB modifications to address errors found in the design
Parts:
- J1, J6: footprint Connector_Molex:Molex_Micro-Fit_3.0_43650-0315_1x03_P3.00mm_Vertical -> CustomFootprints:Molex_Micro-Fit_3.0_43650-0315_1x03_P3.00mm_Vertical
- J2: footprint Connector_Molex:Molex_Micro-Fit_3.0_43650-0415_1x04_P3.00mm_Vertical -> CustomFootprints:Molex_Micro-Fit_3.0_43650-0415_1x04_P3.00mm_Vertical
- J3, J5: footprint Connector_Molex:Molex_Micro-Fit_3.0_43650-0200_1x02_P3.00mm_Horizontal -> CustomFootprints:Molex_Micro-Fit_3.0_43650-0200_1x02_P3.00mm_Horizontal
- J4: footprint Connector_Molex:Molex_Micro-Fit_3.0_43650-0215_1x02_P3.00mm_Vertical -> CustomFootprints:Molex_Micro-Fit_3.0_43650-0215_1x02_P3.00mm_Vertical
Changed lines of the file:
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@@
       (effects (font (size 1.27 1.27)) (justify left))
     )
-    (property "Footprint" "Connector_Molex:Molex_Micro-Fit_3.0_43650-0215_1x02_P3.00mm_Vertical" (at 64.77 104.14 0)
+    (property "Footprint" "CustomFootprints:Molex_Micro-Fit_3.0_43650-0215_1x02_P3.00mm_Vertical" (at 64.77 104.14 0)
       (effects (font (size 1.27 1.27)) hide)
     )
@@
       (effects (font (size 1.27 1.27)) (justify left))
     )
-    (property "Footprint" "Connector_Molex:Molex_Micro-Fit_3.0_43650-0200_1x02_P3.00mm_Horizontal" (at 153.67 50.8 0)
+    (property "Footprint" "CustomFootprints:Molex_Micro-Fit_3.0_43650-0200_1x02_P3.00mm_Horizontal" (at 153.67 50.8 0)
       (effects (font (size 1.27 1.27)) hide)
     )
@@
       (effects (font (size 1.27 1.27)))
     )
-    (property "Footprint" "Connector_Molex:Molex_Micro-Fit_3.0_43650-0315_1x03_P3.00mm_Vertical" (at 64.77 45.72 0)
+    (property "Footprint" "CustomFootprints:Molex_Micro-Fit_3.0_43650-0315_1x03_P3.00mm_Vertical" (at 64.77 45.72 0)
       (effects (font (size 1.27 1.27)) hide)
     )
@@
       (effects (font (size 1.27 1.27)) (justify left))
     )
-    (property "Footprint" "Connector_Molex:Molex_Micro-Fit_3.0_43650-0415_1x04_P3.00mm_Vertical" (at 64.77 59.69 0)
+    (property "Footprint" "CustomFootprints:Molex_Micro-Fit_3.0_43650-0415_1x04_P3.00mm_Vertical" (at 64.77 59.69 0)
       (effects (font (size 1.27 1.27)) hide)
     )
@@
       (effects (font (size 1.27 1.27)) (justify left))
     )
-    (property "Footprint" "Connector_Molex:Molex_Micro-Fit_3.0_43650-0315_1x03_P3.00mm_Vertical" (at 106.68 60.96 0)
+    (property "Footprint" "CustomFootprints:Molex_Micro-Fit_3.0_43650-0315_1x03_P3.00mm_Vertical" (at 106.68 60.96 0)
       (effects (font (size 1.27 1.27)) hide)
     )
@@
       (effects (font (size 1.27 1.27)) (justify left))
     )
-    (property "Footprint" "Connector_Molex:Molex_Micro-Fit_3.0_43650-0200_1x02_P3.00mm_Horizontal" (at 64.77 86.36 0)
-      (effects (font (size 1.27 1.27)) hide)
-    )
+    (property "Footprint" "CustomFootprints:Molex_Micro-Fit_3.0_43650-0200_1x02_P3.00mm_Horizontal" (at 64.77 86.36 0)
+      (effects (font (size 1.27 1.27)) hide)
+    )
