File: Gain1Module/Gain1Module.kicad_pcb (KiCad board)
At the start: 2 copper layers, 56 x 60 mm, 25 parts, among them J1 Low Jack, J2 High Jack, J3 HV, J4 Heater, J5 Signal, J6 Vol, U1 ECC83

Commit message: Change connector footprints to contain 3D models. Make necessary PCB modifications to address errors found in the design
Parts:
- J1, J6: footprint Connector_Molex:Molex_Micro-Fit_3.0_43650-0315_1x03_P3.00mm_Vertical -> CustomFootprints:Molex_Micro-Fit_3.0_43650-0315_1x03_P3.00mm_Vertical
- J2: footprint Connector_Molex:Molex_Micro-Fit_3.0_43650-0415_1x04_P3.00mm_Vertical -> CustomFootprints:Molex_Micro-Fit_3.0_43650-0415_1x04_P3.00mm_Vertical
- J3, J5: footprint Connector_Molex:Molex_Micro-Fit_3.0_43650-0200_1x02_P3.00mm_Horizontal -> CustomFootprints:Molex_Micro-Fit_3.0_43650-0200_1x02_P3.00mm_Horizontal
- J4: footprint Connector_Molex:Molex_Micro-Fit_3.0_43650-0215_1x02_P3.00mm_Vertical -> CustomFootprints:Molex_Micro-Fit_3.0_43650-0215_1x02_P3.00mm_Vertical
Changed lines of the file:
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@@
     )
   )
-  (footprint "Connector_Molex:Molex_Micro-Fit_3.0_43650-0200_1x02_P3.00mm_Horizontal" (layer "F.Cu")
+  (footprint "CustomFootprints:Molex_Micro-Fit_3.0_43650-0200_1x02_P3.00mm_Horizontal" (layer "F.Cu")
     (at 162.05 98.195 -90)
     (descr "Molex Micro-Fit 3.0 Connector System, 43650-0200 (compatible alternatives: 43650-0201, 43650-0202), 2 Pins per row (https://www.molex.com/pdm_docs/sd/436500300_sd.pdf), generated with kicad-footprint-generator")
@@
     (property "ki_keywords" "screw terminal")
     (attr through_hole)
-    (fp_text reference "J3" (at -4.85 -8.13 -180) (layer "F.SilkS")
-        (effects (font (size 1 1) (thickness 0.15)))
-    )
-    (fp_text value "HV" (at 1.5 -6.86 90) (layer "F.Fab")
-        (effects (font (size 1 1) (thickness 0.15)))
-    )
-    (fp_text user "${REFERENCE}" (at 1.5 -8.22 90) (layer "F.Fab")
+    (fp_text reference "J3" (at 1.5 -10.12 -90) (layer "F.SilkS")
+        (effects (font (size 1 1) (thickness 0.15)))
+    )
+    (fp_text value "HV" (at 1.5 3.22 -90) (layer "F.Fab")
+        (effects (font (size 1 1) (thickness 0.15)))
+    )
+    (fp_text user "${REFERENCE}" (at 1.5 -8.22 -90) (layer "F.Fab")
         (effects (font (size 1 1) (thickness 0.15)))
     )
@@
       (scale (xyz 1 1 1))
       (rotate (xyz 0 0 0))
+    )
+    (model "C:/Users/dillo/Downloads/436500200_stp/436500200.stp"
+      (offset (xyz 1.5 8.9 0.5))
+      (scale (xyz 1 1 1))
+      (rotate (xyz 0 0 180))
     )
   )
@@
     )
   )
-  (footprint "Connector_Molex:Molex_Micro-Fit_3.0_43650-0315_1x03_P3.00mm_Vertical" (layer "F.Cu")
+  (footprint "CustomFootprints:Molex_Micro-Fit_3.0_43650-0315_1x03_P3.00mm_Vertical" (layer "F.Cu")
     (at 121.92 69.85 -90)
     (descr "Molex Micro-Fit 3.0 Connector System, 43650-0315 (compatible alternatives: 43650-0316, 43650-0317), 3 Pins per row (http://www.molex.com/pdm_docs/sd/436500215_sd.pdf), generated with kicad-footprint-generator")
@@
     (property "ki_keywords" "screw terminal")
     (attr through_hole)
-    (fp_text reference "J1" (at 3.175 3.175 90) (layer "F.SilkS")
-        (effects (font (size 1 1) (thickness 0.15)))
-    )
-    (fp_text value "Low Jack" (at 3 4.5 90) (layer "F.Fab")
-        (effects (font (size 1 1) (thickness 0.15)))
-    )
-    (fp_text user "${REFERENCE}" (at 3 1.2 90) (layer "F.Fab")
+    (fp_text reference "J1" (at 3 -3.67 -90) (layer "F.SilkS")
+        (effects (font (size 1 1) (thickness 0.15)))
+    )
+    (fp_text value "Low Jack" (at 3 4.5 -90) (layer "F.Fab")
+        (effects (font (size 1 1) (thickness 0.15)))
+    )
+    (fp_text user "${REFERENCE}" (at 3 1.2 -90) (layer "F.Fab")
         (effects (font (size 1 1) (thickness 0.15)))
     )
@@
       (rotate (xyz 0 0 0))
     )
-  )
-  (footprint "Connector_Molex:Molex_Micro-Fit_3.0_43650-0315_1x03_P3.00mm_Vertical" (layer "F.Cu")
+    (model "C:/Users/dillo/Downloads/436500315_stp/436500315.stp"
+      (offset (xyz 3 1.9 10))
+      (scale (xyz 1 1 1))
+      (rotate (xyz 90 0 180))
+    )
+  )
+  (footprint "CustomFootprints:Molex_Micro-Fit_3.0_43650-0315_1x03_P3.00mm_Vertical" (layer "F.Cu")
     (at 138.43 72.04 90)
     (descr "Molex Micro-Fit 3.0 Connector System, 43650-0315 (compatible alternatives: 43650-0316, 43650-0317), 3 Pins per row (http://www.molex.com/pdm_docs/sd/436500215_sd.pdf), generated with kicad-footprint-generator")
@@
     (property "ki_keywords" "screw terminal")
     (attr through_hole)
-    (fp_text reference "J6" (at 10.445 0 180) (layer "F.SilkS")
+    (fp_text reference "J6" (at 3 -3.67 90) (layer "F.SilkS")
         (effects (font (size 1 1) (thickness 0.15)))
     )
@@
       (rotate (xyz 0 0 0))
     )
+    (model "C:/Users/dillo/Downloads/436500315_stp/436500315.stp"
+      (offset (xyz 3 1.9 10))
+      (scale (xyz 1 1 1))
+      (rotate (xyz 90 0 180))
+    )
   )
   (footprint "Resistor_THT:R_Axial_DIN0309_L9.0mm_D3.2mm_P12.70mm_Horizontal" (layer "F.Cu")
@@
     (pad "" np_thru_hole circle (at 0 0) (size 2.5 2.5) (drill 2.5) (layers "F&B.Cu" "*.Mask"))
   )
-  (footprint "Connector_Molex:Molex_Micro-Fit_3.0_43650-0215_1x02_P3.00mm_Vertical" (layer "F.Cu")
+  (footprint "CustomFootprints:Molex_Micro-Fit_3.0_43650-0215_1x02_P3.00mm_Vertical" (layer "F.Cu")
     (at 144.09 84.915 -90)
     (descr "Molex Micro-Fit 3.0 Connector System, 43650-0215 (compatible alternatives: 43650-0216, 43650-0217), 2 Pins per row (http://www.molex.com/pdm_docs/sd/436500215_sd.pdf), generated with kicad-footprint-generator")
@@
     (property "ki_keywords" "screw terminal")
     (attr through_hole)
-    (fp_text reference "J4" (at 1.5 -3.67 90) (layer "F.SilkS")
-        (effects (font (size 1 1) (thickness 0.15)))
-    )
-    (fp_text value "Heater" (at 1.5 4.5 90) (layer "F.Fab")
-        (effects (font (size 1 1) (thickness 0.15)))
-    )
-    (fp_text user "${REFERENCE}" (at 1.5 1.2 90) (layer "F.Fab")
+    (fp_text reference "J4" (at 1.5 -3.67 -90) (layer "F.SilkS")
+        (effects (font (size 1 1) (thickness 0.15)))
+    )
+    (fp_text value "Heater" (at 1.5 4.5 -90) (layer "F.Fab")
+        (effects (font (size 1 1) (thickness 0.15)))
+    )
+    (fp_text user "${REFERENCE}" (at 1.5 1.2 -90) (layer "F.Fab")
         (effects (font (size 1 1) (thickness 0.15)))
     )
@@
       (rotate (xyz 0 0 0))
     )
-  )
-  (footprint "Connector_Molex:Molex_Micro-Fit_3.0_43650-0200_1x02_P3.00mm_Horizontal" (layer "F.Cu")
+    (model "C:/Users/dillo/Downloads/436500215_stp/436500215.stp"
+      (offset (xyz 1.5 1.9 10))
+      (scale (xyz 1 1 1))
+      (rotate (xyz 90 0 180))
+    )
+  )
+  (footprint "CustomFootprints:Molex_Micro-Fit_3.0_43650-0200_1x02_P3.00mm_Horizontal" (layer "F.Cu")
     (at 162.05 71.525 -90)
     (descr "Molex Micro-Fit 3.0 Connector System, 43650-0200 (compatible alternatives: 43650-0201, 43650-0202), 2 Pins per row (https://www.molex.com/pdm_docs/sd/436500300_sd.pdf), generated with kicad-footprint-generator")
@@
     (property "ki_keywords" "screw terminal")
     (attr through_hole)
-    (fp_text reference "J5" (at 7.85 -8.13 -180) (layer "F.SilkS")
-        (effects (font (size 1 1) (thickness 0.15)))
-    )
-    (fp_text value "Signal" (at 1.5 -6.86 90) (layer "F.Fab")
-        (effects (font (size 1 1) (thickness 0.15)))
-    )
-    (fp_text user "${REFERENCE}" (at 1.5 -8.22 90) (layer "F.Fab")
+    (fp_text reference "J5" (at 1.5 -10.12 -90) (layer "F.SilkS")
+        (effects (font (size 1 1) (thickness 0.15)))
+    )
+    (fp_text value "Signal" (at 1.5 3.22 -90) (layer "F.Fab")
+        (effects (font (size 1 1) (thickness 0.15)))
+    )
+    (fp_text user "${REFERENCE}" (at 1.5 -8.22 -90) (layer "F.Fab")
         (effects (font (size 1 1) (thickness 0.15)))
     )
@@
       (scale (xyz 1 1 1))
       (rotate (xyz 0 0 0))
+    )
+    (model "C:/Users/dillo/Downloads/436500200_stp/436500200.stp"
+      (offset (xyz 1.5 8.9 0.5))
+      (scale (xyz 1 1 1))
+      (rotate (xyz 0 0 180))
     )
   )
@@
     )
   )
-  (footprint "Connector_Molex:Molex_Micro-Fit_3.0_43650-0415_1x04_P3.00mm_Vertical" (layer "F.Cu")
+  (footprint "CustomFootprints:Molex_Micro-Fit_3.0_43650-0415_1x04_P3.00mm_Vertical" (layer "F.Cu")
     (at 126.365 103.395 -90)
     (descr "Molex Micro-Fit 3.0 Connector System, 43650-0415 (compatible alternatives: 43650-0416, 43650-0417), 4 Pins per row (http://www.molex.com/pdm_docs/sd/436500215_sd.pdf), generated with kicad-footprint-generator")
@@
     (property "ki_keywords" "screw terminal")
     (attr through_hole)
-    (fp_text reference "J2" (at 4.5 3.175 90) (layer "F.SilkS")
-        (effects (font (size 1 1) (thickness 0.15)))
-    )
-    (fp_text value "High Jack" (at 4.5 4.5 90) (layer "F.Fab")
-        (effects (font (size 1 1) (thickness 0.15)))
-    )
-    (fp_text user "${REFERENCE}" (at 4.5 1.2 90) (layer "F.Fab")
+    (fp_text reference "J2" (at 4.5 -3.67 -90) (layer "F.SilkS")
+        (effects (font (size 1 1) (thickness 0.15)))
+    )
+    (fp_text value "High Jack" (at 4.5 4.5 -90) (layer "F.Fab")
+        (effects (font (size 1 1) (thickness 0.15)))
+    )
+    (fp_text user "${REFERENCE}" (at 4.5 1.2 -90) (layer "F.Fab")
         (effects (font (size 1 1) (thickness 0.15)))
     )
@@
       (rotate (xyz 0 0 0))
     )
-  )
+    (model "C:/Users/dillo/Downloads/436500415_stp/436500415.stp"
+      (offset (xyz 4.5 1.9 10))
+      (scale (xyz 1 1 1))
+      (rotate (xyz 90 0 180))
+    )
+  )

Commit message: Standardized hole size across all boards
Parts:
- removed the REF** at (118.5, 59.4)
- removed the REF** at (168.5, 59.4)
- removed the REF** at (118.5, 113.4)
- removed the REF** at (168.5, 113.4)
- added REF**: MountingHole_2.7mm_M2.5, MountingHole:MountingHole_2.7mm_M2.5, F.Cu at (168.5, 59.4)
- added REF**: MountingHole_2.7mm_M2.5_Pad, MountingHole:MountingHole_2.7mm_M2.5_Pad, F.Cu at (118.5, 113.4)
- added REF**: MountingHole_2.7mm_M2.5, MountingHole:MountingHole_2.7mm_M2.5, F.Cu at (168.5, 113.4)
- added REF**: MountingHole_2.7mm_M2.5, MountingHole:MountingHole_2.7mm_M2.5, F.Cu at (118.5, 59.4)
Routing:
- net GND1: track 24.2 -> 15.4 mm
Changed lines of the file:
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@@
     )
   )
-  (footprint "MountingHole:MountingHole_2.5mm" (layer "F.Cu")
-    (at 118.51 59.36)
-    (descr "Mounting Hole 2.5mm, no annular")
-    (tags "mounting hole 2.5mm no annular")
+  (footprint "MountingHole:MountingHole_2.7mm_M2.5" (layer "F.Cu")
+    (at 168.51 59.36)
+    (descr "Mounting Hole 2.7mm, no annular, M2.5")
+    (tags "mounting hole 2.7mm no annular m2.5")
     (attr exclude_from_pos_files exclude_from_bom)
-    (fp_text reference "REF**" (at 0 -3.5) (layer "F.SilkS") hide
-        (effects (font (size 1 1) (thickness 0.15)))
-    )
-    (fp_text value "MountingHole_2.5mm" (at 0 3.5) (layer "F.Fab") hide
+    (fp_text reference "REF**" (at 0 -3.7) (layer "F.SilkS") hide
+        (effects (font (size 1 1) (thickness 0.15)))
+    )
+    (fp_text value "MountingHole_2.7mm_M2.5" (at 0 3.7) (layer "F.Fab") hide
         (effects (font (size 1 1) (thickness 0.15)))
     )
@@
         (effects (font (size 1 1) (thickness 0.15)))
     )
-    (fp_circle (center 0 0) (end 2.5 0)
+    (fp_circle (center 0 0) (end 2.7 0)
       (stroke (width 0.15) (type solid)) (fill none) (layer "Cmts.User"))
-    (fp_circle (center 0 0) (end 2.75 0)
+    (fp_circle (center 0 0) (end 2.95 0)
       (stroke (width 0.05) (type solid)) (fill none) (layer "F.CrtYd"))
-    (pad "" np_thru_hole circle (at 0 0) (size 2.5 2.5) (drill 2.5) (layers "F&B.Cu" "*.Mask"))
+    (pad "" np_thru_hole circle (at 0 0) (size 2.7 2.7) (drill 2.7) (layers "*.Cu" "*.Mask"))
   )
   (footprint "Capacitor_THT:C_Rect_L13.0mm_W4.0mm_P10.00mm_FKS3_FKP3_MKS4" (layer "F.Cu")
@@
       (rotate (xyz 0 0 0))
     )
+  )
+  (footprint "MountingHole:MountingHole_2.7mm_M2.5_Pad" (layer "F.Cu")
+    (at 118.51 113.36)
+    (descr "Mounting Hole 2.7mm, M2.5")
+    (tags "mounting hole 2.7mm m2.5")
+    (attr exclude_from_pos_files exclude_from_bom)
+    (fp_text reference "REF**" (at 0 -3.7) (layer "F.SilkS") hide
+        (effects (font (size 1 1) (thickness 0.15)))
+    )
+    (fp_text value "MountingHole_2.7mm_M2.5_Pad" (at 0 3.7) (layer "F.Fab") hide
+        (effects (font (size 1 1) (thickness 0.15)))
+    )
+    (fp_text user "${REFERENCE}" (at 0 0) (layer "F.Fab")
+        (effects (font (size 1 1) (thickness 0.15)))
+    )
+    (fp_circle (center 0 0) (end 2.7 0)
+      (stroke (width 0.15) (type solid)) (fill none) (layer "Cmts.User"))
+    (fp_circle (center 0 0) (end 2.95 0)
+      (stroke (width 0.05) (type solid)) (fill none) (layer "F.CrtYd"))
+    (pad "1" thru_hole circle (at 0 0) (size 5.4 5.4) (drill 2.7) (layers "*.Cu" "*.Mask")
+      (net 4 "GND"))
   )
   (footprint "CustomFootprints:FG26 Cap" (layer "F.Cu")
@@
     )
   )
+  (footprint "MountingHole:MountingHole_2.7mm_M2.5" (layer "F.Cu")
+    (at 168.51 113.36)
+    (descr "Mounting Hole 2.7mm, no annular, M2.5")
+    (tags "mounting hole 2.7mm no annular m2.5")
+    (attr exclude_from_pos_files exclude_from_bom)
+    (fp_text reference "REF**" (at 0 -3.7) (layer "F.SilkS") hide
+        (effects (font (size 1 1) (thickness 0.15)))
+    )
+    (fp_text value "MountingHole_2.7mm_M2.5" (at 0 3.7) (layer "F.Fab") hide
+        (effects (font (size 1 1) (thickness 0.15)))
+    )
+    (fp_text user "${REFERENCE}" (at 0 0) (layer "F.Fab")
+        (effects (font (size 1 1) (thickness 0.15)))
+    )
+    (fp_circle (center 0 0) (end 2.7 0)
+      (stroke (width 0.15) (type solid)) (fill none) (layer "Cmts.User"))
+    (fp_circle (center 0 0) (end 2.95 0)
+      (stroke (width 0.05) (type solid)) (fill none) (layer "F.CrtYd"))
+    (pad "" np_thru_hole circle (at 0 0) (size 2.7 2.7) (drill 2.7) (layers "*.Cu" "*.Mask"))
+  )
   (footprint "Capacitor_THT:CP_Radial_D13.0mm_P5.00mm" (layer "F.Cu")
     (at 154.94 106.76 -90)
@@
     )
   )
-  (footprint "MountingHole:MountingHole_2.5mm" (layer "F.Cu")
-    (at 168.51 59.36)
-    (descr "Mounting Hole 2.5mm, no annular")
-    (tags "mounting hole 2.5mm no annular")
+  (footprint "MountingHole:MountingHole_2.7mm_M2.5" (layer "F.Cu")
+    (at 118.51 59.36)
+    (descr "Mounting Hole 2.7mm, no annular, M2.5")
+    (tags "mounting hole 2.7mm no annular m2.5")
     (attr exclude_from_pos_files exclude_from_bom)
-    (fp_text reference "REF**" (at 0 -3.5) (layer "F.SilkS") hide
-        (effects (font (size 1 1) (thickness 0.15)))
-    )
-    (fp_text value "MountingHole_2.5mm" (at 0 3.5) (layer "F.Fab") hide
+    (fp_text reference "REF**" (at 0 -3.7) (layer "F.SilkS") hide
+        (effects (font (size 1 1) (thickness 0.15)))
+    )
+    (fp_text value "MountingHole_2.7mm_M2.5" (at 0 3.7) (layer "F.Fab") hide
         (effects (font (size 1 1) (thickness 0.15)))
     )
@@
         (effects (font (size 1 1) (thickness 0.15)))
     )
-    (fp_circle (center 0 0) (end 2.5 0)
+    (fp_circle (center 0 0) (end 2.7 0)
       (stroke (width 0.15) (type solid)) (fill none) (layer "Cmts.User"))
-    (fp_circle (center 0 0) (end 2.75 0)
+    (fp_circle (center 0 0) (end 2.95 0)
       (stroke (width 0.05) (type solid)) (fill none) (layer "F.CrtYd"))
-    (pad "" np_thru_hole circle (at 0 0) (size 2.5 2.5) (drill 2.5) (layers "F&B.Cu" "*.Mask"))
+    (pad "" np_thru_hole circle (at 0 0) (size 2.7 2.7) (drill 2.7) (layers "*.Cu" "*.Mask"))
   )
   (footprint "CustomFootprints:Molex_Micro-Fit_3.0_43650-0215_1x02_P3.00mm_Vertical" (layer "F.Cu")
@@
       (rotate (xyz 0 0 180))
     )
-  )
-  (footprint "MountingHole:MountingHole_2.5mm_Pad" (layer "F.Cu")
-    (at 118.51 113.36)
-    (descr "Mounting Hole 2.5mm")
-    (tags "mounting hole 2.5mm")
-    (attr exclude_from_pos_files exclude_from_bom)
-    (fp_text reference "REF**" (at 0 -3.5) (layer "F.SilkS") hide
-        (effects (font (size 1 1) (thickness 0.15)))
-    )
-    (fp_text value "MountingHole_2.5mm_Pad" (at 0 3.5) (layer "F.Fab") hide
-        (effects (font (size 1 1) (thickness 0.15)))
-    )
-    (fp_text user "${REFERENCE}" (at 0 0) (layer "F.Fab")
-        (effects (font (size 1 1) (thickness 0.15)))
-    )
-    (fp_circle (center 0 0) (end 2.5 0)
-      (stroke (width 0.15) (type solid)) (fill none) (layer "Cmts.User"))
-    (fp_circle (center 0 0) (end 2.75 0)
-      (stroke (width 0.05) (type solid)) (fill none) (layer "F.CrtYd"))
-    (pad "1" thru_hole circle (at 0 0) (size 5 5) (drill 2.5) (layers "*.Cu" "*.Mask")
-      (net 4 "GND"))
   )
   (footprint "Capacitor_THT:C_Rect_L10.0mm_W4.0mm_P7.50mm_MKS4" (layer "F.Cu")
@@
       (rotate (xyz 90 0 180))
     )
-  )
-  (footprint "MountingHole:MountingHole_2.5mm_Pad" (layer "F.Cu")
-    (at 168.51 113.36)
-    (descr "Mounting Hole 2.5mm")
-    (tags "mounting hole 2.5mm")
-    (attr exclude_from_pos_files exclude_from_bom)
-    (fp_text reference "REF**" (at 0 -3.5) (layer "F.SilkS") hide
-        (effects (font (size 1 1) (thickness 0.15)))
-    )
-    (fp_text value "MountingHole_2.5mm_Pad" (at 0 3.5) (layer "F.Fab") hide
-        (effects (font (size 1 1) (thickness 0.15)))
-    )
-    (fp_text user "${REFERENCE}" (at 0 0) (layer "F.Fab")
-        (effects (font (size 1 1) (thickness 0.15)))
-    )
-    (fp_circle (center 0 0) (end 2.5 0)
-      (stroke (width 0.15) (type solid)) (fill none) (layer "Cmts.User"))
-    (fp_circle (center 0 0) (end 2.75 0)
-      (stroke (width 0.05) (type solid)) (fill none) (layer "F.CrtYd"))
-    (pad "1" thru_hole circle (at 0 0) (size 5 5) (drill 2.5) (layers "*.Cu" "*.Mask")
-      (net 11 "GND1"))
   )
   (footprint "CustomFootprints:BELTON_VT9-PT" (layer "B.Cu")
@@
   (segment (start 128.15 112.395) (end 132.08 108.465) (width 2) (layer "B.Cu") (net 4))
   (segment (start 149.225 60.96) (end 149.225 62.23) (width 2) (layer "B.Cu") (net 4))
+  (segment (start 126.365 112.395) (end 119.475 112.395) (width 2) (layer "B.Cu") (net 4))
   (segment (start 134.62 99.695) (end 136.525 97.79) (width 2) (layer "B.Cu") (net 4))
   (segment (start 146.05 93.98) (end 146.05 94.615) (width 2) (layer "B.Cu") (net 4))
@@
   (segment (start 136.525 82.55) (end 139.7 82.55) (width 2) (layer "B.Cu") (net 4))
   (segment (start 139.7 82.55) (end 143.111 79.139) (width 2) (layer "B.Cu") (net 4))
+  (segment (start 119.475 112.395) (end 118.51 113.36) (width 2) (layer "B.Cu") (net 4))
   (segment (start 142.25627 66.04) (end 146.98 70.76373) (width 2) (layer "B.Cu") (net 4))
   (segment (start 145.415 93.98) (end 146.05 94.615) (width 2) (layer "B.Cu") (net 4))
@@
   (segment (start 155.665 77.453292) (end 151.026 82.092292) (width 2) (layer "B.Cu") (net 4))
   (segment (start 130.81 74.270001) (end 130.81 76.835) (width 2) (layer "B.Cu") (net 4))
-  (segment (start 126.365 112.395) (end 120.015 112.395) (width 2) (layer "B.Cu") (net 4))
   (segment (start 158.593292 74.525) (end 162.05 74.525) (width 2) (layer "B.Cu") (net 4))
   (segment (start 148.658592 91.371408) (end 146.05 93.98) (width 2) (layer "B.Cu") (net 4))
@@
   (segment (start 136.525 97.79) (end 138.43 97.79) (width 2) (layer "B.Cu") (net 4))
   (segment (start 143.111 79.139) (end 146.98 79.139) (width 2) (layer "B.Cu") (net 4))
-  (segment (start 120.015 112.395) (end 118.745 113.665) (width 2) (layer "B.Cu") (net 4))
   (segment (start 152.4 65.405) (end 155.665 68.67) (width 2) (layer "B.Cu") (net 4))
   (segment (start 146.685 100.33) (end 146.05 100.965) (width 2) (layer "B.Cu") (net 4))
@@
   (segment (start 162.05 101.195) (end 162.05 104.159785) (width 2) (layer "B.Cu") (net 11))
   (segment (start 158.115 111.76) (end 154.94 111.76) (width 2) (layer "B.Cu") (net 11))
-  (segment (start 162.05 107.44) (end 168.275 113.665) (width 2) (layer "B.Cu") (net 11))
   (segment (start 162.05 104.159785) (end 162.05 107.44) (width 2) (layer "B.Cu") (net 11))
   (segment (start 162.05 107.44) (end 162.05 107.825) (width 2) (layer "B.Cu") (net 11))
