File: Gain2Module/Gain2Module.kicad_sch (KiCad schematic)
At the start: 15 parts, among them J1 SigIn, J2 SigOut, J3 Heater, J4 HeaterOut, J5 HV, J6 HVOut, U1 ECC83

Commit message: Change connector footprints to contain 3D models. Make necessary PCB modifications to address errors found in the design
Parts:
- J1, J2, J5, J6: footprint Connector_Molex:Molex_Micro-Fit_3.0_43650-0200_1x02_P3.00mm_Horizontal -> CustomFootprints:Molex_Micro-Fit_3.0_43650-0200_1x02_P3.00mm_Horizontal
- J3, J4: footprint Connector_Molex:Molex_Micro-Fit_3.0_43650-0215_1x02_P3.00mm_Vertical -> CustomFootprints:Molex_Micro-Fit_3.0_43650-0215_1x02_P3.00mm_Vertical
Changed lines of the file:
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@@
       (effects (font (size 1.27 1.27)) (justify left))
     )
-    (property "Footprint" "Connector_Molex:Molex_Micro-Fit_3.0_43650-0200_1x02_P3.00mm_Horizontal" (at 95.25 99.06 0)
+    (property "Footprint" "CustomFootprints:Molex_Micro-Fit_3.0_43650-0200_1x02_P3.00mm_Horizontal" (at 95.25 99.06 0)
       (effects (font (size 1.27 1.27)) hide)
     )
@@
       (effects (font (size 1.27 1.27)) (justify left))
     )
-    (property "Footprint" "Connector_Molex:Molex_Micro-Fit_3.0_43650-0215_1x02_P3.00mm_Vertical" (at 132.08 143.51 0)
+    (property "Footprint" "CustomFootprints:Molex_Micro-Fit_3.0_43650-0215_1x02_P3.00mm_Vertical" (at 132.08 143.51 0)
       (effects (font (size 1.27 1.27)) hide)
     )
@@
       (effects (font (size 1.27 1.27)) (justify left))
     )
-    (property "Footprint" "Connector_Molex:Molex_Micro-Fit_3.0_43650-0200_1x02_P3.00mm_Horizontal" (at 106.68 54.61 0)
+    (property "Footprint" "CustomFootprints:Molex_Micro-Fit_3.0_43650-0200_1x02_P3.00mm_Horizontal" (at 106.68 54.61 0)
       (effects (font (size 1.27 1.27)) hide)
     )
@@
       (effects (font (size 1.27 1.27)) (justify left))
     )
-    (property "Footprint" "Connector_Molex:Molex_Micro-Fit_3.0_43650-0215_1x02_P3.00mm_Vertical" (at 106.68 140.97 0)
+    (property "Footprint" "CustomFootprints:Molex_Micro-Fit_3.0_43650-0215_1x02_P3.00mm_Vertical" (at 106.68 140.97 0)
       (effects (font (size 1.27 1.27)) hide)
     )
@@
       (effects (font (size 1.27 1.27)) (justify left))
     )
-    (property "Footprint" "Connector_Molex:Molex_Micro-Fit_3.0_43650-0200_1x02_P3.00mm_Horizontal" (at 134.62 57.15 0)
+    (property "Footprint" "CustomFootprints:Molex_Micro-Fit_3.0_43650-0200_1x02_P3.00mm_Horizontal" (at 134.62 57.15 0)
       (effects (font (size 1.27 1.27)) hide)
     )
@@
       (effects (font (size 1.27 1.27)) (justify left))
     )
-    (property "Footprint" "Connector_Molex:Molex_Micro-Fit_3.0_43650-0200_1x02_P3.00mm_Horizontal" (at 160.02 106.68 0)
-      (effects (font (size 1.27 1.27)) hide)
-    )
+    (property "Footprint" "CustomFootprints:Molex_Micro-Fit_3.0_43650-0200_1x02_P3.00mm_Horizontal" (at 160.02 106.68 0)
+      (effects (font (size 1.27 1.27)) hide)
+    )
