File: PowerAmpModule/PowerAmpModule.kicad_sch (KiCad schematic)
At the start: 16 parts, among them J1 Signal, J2 Power, J3 SignalOut, J4 Heater, J5 HeaterOut, J6 PowerOut, J7 Inductor, U1 6V6, U2 6V6

Commit message: Standardized hole size across all boards
Parts:
- J1: footprint Connector_Molex:Molex_Micro-Fit_3.0_43650-0300_1x03_P3.00mm_Horizontal -> CustomFootprints:Molex_Micro-Fit_3.0_43650-0300_1x03_P3.00mm_Horizontal
- J2, J3: footprint Connector_Molex:Molex_Micro-Fit_3.0_43650-0315_1x03_P3.00mm_Vertical -> CustomFootprints:Molex_Micro-Fit_3.0_43650-0315_1x03_P3.00mm_Vertical
- J4, J5: footprint Connector_Molex:Molex_Micro-Fit_3.0_43650-0215_1x02_P3.00mm_Vertical -> CustomFootprints:Molex_Micro-Fit_3.0_43045-0412_2x02_P3.00mm_Vertical
- J6: footprint Connector_Molex:Molex_Micro-Fit_3.0_43650-0200_1x02_P3.00mm_Horizontal -> CustomFootprints:Molex_Micro-Fit_3.0_43650-0200_1x02_P3.00mm_Horizontal
- J7: footprint Connector_Molex:Molex_Micro-Fit_3.0_43650-0215_1x02_P3.00mm_Vertical -> CustomFootprints:Molex_Micro-Fit_3.0_43650-0215_1x02_P3.00mm_Vertical
Changed lines of the file:
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@@
       (effects (font (size 1.27 1.27)) (justify left))
     )
-    (property "Footprint" "Connector_Molex:Molex_Micro-Fit_3.0_43650-0215_1x02_P3.00mm_Vertical" (at 154.94 143.51 0)
+    (property "Footprint" "CustomFootprints:Molex_Micro-Fit_3.0_43045-0412_2x02_P3.00mm_Vertical" (at 154.94 143.51 0)
       (effects (font (size 1.27 1.27)) hide)
     )
@@
       (effects (font (size 1.27 1.27)) (justify left))
     )
-    (property "Footprint" "Connector_Molex:Molex_Micro-Fit_3.0_43650-0315_1x03_P3.00mm_Vertical" (at 116.84 58.42 0)
+    (property "Footprint" "CustomFootprints:Molex_Micro-Fit_3.0_43650-0315_1x03_P3.00mm_Vertical" (at 116.84 58.42 0)
       (effects (font (size 1.27 1.27)) hide)
     )
@@
       (effects (font (size 1.27 1.27)) (justify right))
     )
-    (property "Footprint" "Connector_Molex:Molex_Micro-Fit_3.0_43650-0215_1x02_P3.00mm_Vertical" (at 128.27 50.8 0)
+    (property "Footprint" "CustomFootprints:Molex_Micro-Fit_3.0_43650-0215_1x02_P3.00mm_Vertical" (at 128.27 50.8 0)
       (effects (font (size 1.27 1.27)) hide)
     )
@@
       (effects (font (size 1.27 1.27)) (justify left))
     )
-    (property "Footprint" "Connector_Molex:Molex_Micro-Fit_3.0_43650-0215_1x02_P3.00mm_Vertical" (at 116.84 143.51 0)
+    (property "Footprint" "CustomFootprints:Molex_Micro-Fit_3.0_43045-0412_2x02_P3.00mm_Vertical" (at 116.84 143.51 0)
       (effects (font (size 1.27 1.27)) hide)
     )
@@
       (effects (font (size 1.27 1.27)) (justify left))
     )
-    (property "Footprint" "Connector_Molex:Molex_Micro-Fit_3.0_43650-0300_1x03_P3.00mm_Horizontal" (at 95.25 95.25 0)
+    (property "Footprint" "CustomFootprints:Molex_Micro-Fit_3.0_43650-0300_1x03_P3.00mm_Horizontal" (at 95.25 95.25 0)
       (effects (font (size 1.27 1.27)) hide)
     )
@@
       (effects (font (size 1.27 1.27)) (justify left))
     )
-    (property "Footprint" "Connector_Molex:Molex_Micro-Fit_3.0_43650-0200_1x02_P3.00mm_Horizontal" (at 149.86 55.88 0)
+    (property "Footprint" "CustomFootprints:Molex_Micro-Fit_3.0_43650-0200_1x02_P3.00mm_Horizontal" (at 149.86 55.88 0)
       (effects (font (size 1.27 1.27)) hide)
     )
@@
       (effects (font (size 1.27 1.27)) (justify left))
     )
-    (property "Footprint" "Connector_Molex:Molex_Micro-Fit_3.0_43650-0315_1x03_P3.00mm_Vertical" (at 165.1 88.9 0)
-      (effects (font (size 1.27 1.27)) hide)
-    )
+    (property "Footprint" "CustomFootprints:Molex_Micro-Fit_3.0_43650-0315_1x03_P3.00mm_Vertical" (at 165.1 88.9 0)
+      (effects (font (size 1.27 1.27)) hide)
+    )
